Commit message: Update

File: ros_1/catkin_ws/src/my_package/urdf/robot.urdf.xacro (robot description, xacro)
@@ -3,6 +3,6 @@
     <xacro:include filename="utils.xacro"/>
     <xacro:include filename="robot_core_v0.xacro"/>
-    <xacro:include filename="table.xacro"/>
-    <xacro:include filename="camera.xacro"/>
+    <xacro:include filename="table_old.xacro"/>
+    <xacro:include filename="camera_old.xacro"/>
     <xacro:include filename="person.xacro"/>
     <xacro:include filename="example_gazebo.xacro"/>

File: ros_1/catkin_ws/src/my_package/urdf/table_old.xacro (robot description, xacro)
@@ -53,5 +53,4 @@
 </xacro:macro>
 <xacro:place_legs pos_x="${o_x}" pos_y="${o_y}" table_x="${table_x}" table_y="${table_y}" />
-<link name="world" />
 <link name="table">
     <visual>
