Commit message: Update

File: ros_1/catkin_ws/src/my_package/urdf/panda_arm_hand.urdf.xacro (robot description, xacro)
@@ -12,3 +12,4 @@
     <xacro:panda_control arm_id="panda"/>
   <!-- </xacro:if> -->
+  <!-- <xacro:include filename="$(find my_package)/urdf/person_new_2.xacro"/> -->
 </robot>

File: ros_1/catkin_ws/src/my_package/urdf/person_new.xacro (robot description, xacro)
@@ -15,5 +15,6 @@
     <visual>
       <geometry>
-        <mesh filename="/usr/share/gazebo-11/media/models/stand.dae" scale="0.5 0.5 0.5"/>
+        <!-- <mesh filename="/usr/share/gazebo-11/media/models/stand.dae" scale="0.5 0.5 0.5"/> -->
+        <mesh filename="package://my_package/meshes/stand.dae" scale="0.5 0.5 0.5"/>
       </geometry>
       <origin xyz="0 0 ${person_height/2}" rpy="0 0 0"/>

File: ros_1/catkin_ws/src/my_package/urdf/person_new_2.xacro (robot description, xacro)
@@ -11,5 +11,5 @@
     </inertial>
   </xacro:macro>
-    <link name="world" />
+    <!-- <link name="world" /> -->
     <link name="x_axis_link">
         <visual>
@@ -38,5 +38,5 @@
     <child link="x_axis_link"/>
     <origin xyz="0 0 0.01" />
-    <dynamics damping="1.0"/>
+    <dynamics damping="10.0"/>
   </joint>
   <transmission name="person_tran1">
@@ -76,5 +76,5 @@
   <child link="y_axis_link"/>
   <origin xyz="0 0 0.01" />
-  <dynamics damping="1.0"/>
+  <dynamics damping="10.0"/>
 </joint>
 <transmission name="person_tran2">
@@ -120,9 +120,3 @@
     <origin xyz="0 0 0.025" />
   </joint>
-  <gazebo>
-    <plugin name="gazebo_ros_control" filename="libgazebo_ros_control.so">
-      <robotNamespace>/person</robotNamespace>
-      <robotParam>/person_description</robotParam>
-    </plugin>
-  </gazebo>
 </robot>
