Commit message: Update

File: ros_1/catkin_ws/src/my_package/urdf/panda_arm.xacro (robot description, xacro)
@@ -220,5 +220,7 @@
     <link name="${arm_id}_link8"/>
     <joint name="${arm_id}_joint8" type="fixed">
-      <origin rpy="0 0 0" xyz="0 0 0.107"/>
+      <!-- <origin rpy="0 0 0" xyz="0 0 0.107"/> -->
+      <!-- <origin rpy="0 0 0" xyz="0 0 0.055"/> -->
+      <origin rpy="0 0 0" xyz="0 0 $(arg attach_offset)"/>
       <parent link="${arm_id}_link7"/>
       <child link="${arm_id}_link8"/>

File: ros_1/catkin_ws/src/my_package/urdf/panda_arm_hand.urdf.xacro (robot description, xacro)
@@ -1,4 +1,5 @@
 <?xml version="1.0" encoding="utf-8"?>
 <robot xmlns:xacro="http://www.ros.org/wiki/xacro" name="panda">
+  <xacro:arg name="attach_offset" default="0.107" />
   <xacro:include filename="$(find my_package)/urdf/panda_arm.xacro"/>
   <xacro:include filename="$(find my_package)/urdf/hand.xacro"/>

Commit message: Update

File: ros_1/catkin_ws/src/my_package/urdf/panda_arm.xacro (robot description, xacro)
@@ -222,5 +222,5 @@
       <!-- <origin rpy="0 0 0" xyz="0 0 0.107"/> -->
       <!-- <origin rpy="0 0 0" xyz="0 0 0.055"/> -->
-      <origin rpy="0 0 0" xyz="0 0 $(arg attach_offset)"/>
+      <origin rpy="0 0 0" xyz="0 0 $(arg joint8_offset)"/>
       <parent link="${arm_id}_link7"/>
       <child link="${arm_id}_link8"/>

Commit message: Update

File: ros_1/catkin_ws/src/my_package/urdf/panda_arm.xacro (robot description, xacro)
@@ -12,10 +12,4 @@
     <dynamics damping="${joint_damping}"/>
   </joint>
-      <joint name="${arm_id}_joint_${connected_to}" type="fixed">
-        <parent link="${connected_to}"/>
-        <child link="${arm_id}_link0"/>
-        <origin rpy="${rpy}" xyz="${xyz}"/>
-        <dynamics damping="${joint_damping}"/>
-      </joint>
     </xacro:unless>
     <link name="${arm_id}_link0">

Commit message: Update

File: ros_1/catkin_ws/src/my_package/urdf/panda_arm.xacro (robot description, xacro)
@@ -214,7 +214,5 @@
     <link name="${arm_id}_link8"/>
     <joint name="${arm_id}_joint8" type="fixed">
-      <!-- <origin rpy="0 0 0" xyz="0 0 0.107"/> -->
-      <!-- <origin rpy="0 0 0" xyz="0 0 0.055"/> -->
-      <origin rpy="0 0 0" xyz="0 0 $(arg joint8_offset)"/>
+      <origin rpy="0 0 0" xyz="0 0 0.107"/>
       <parent link="${arm_id}_link7"/>
       <child link="${arm_id}_link8"/>

File: ros_1/catkin_ws/src/my_package/urdf/panda_arm_hand.urdf.xacro (robot description, xacro)
@@ -1,5 +1,4 @@
 <?xml version="1.0" encoding="utf-8"?>
 <robot xmlns:xacro="http://www.ros.org/wiki/xacro" name="panda">
-  <xacro:arg name="joint8_offset" default="0.107" />
   <!-- <xacro:arg name="gazebo" default="false" /> -->
   <xacro:include filename="$(find my_package)/urdf/panda_arm.xacro"/>

Commit message: Update

File: ros_1/catkin_ws/src/my_package/urdf/panda_arm.xacro (robot description, xacro)
@@ -9,5 +9,5 @@
     <parent link="world" />
     <child link="${arm_id}_link0" />
-    <origin xyz="0.0 0.0 0.0" rpy="0.0 0.0 0.0" />
+    <origin xyz="0.0 0.0 0.4" rpy="0.0 0.0 0.0" />
     <dynamics damping="${joint_damping}"/>
   </joint>

File: ros_1/catkin_ws/src/my_package/urdf/person_new_3.xacro (robot description, xacro)
@@ -11,5 +11,5 @@
     </inertial>
   </xacro:macro>
-    <link name="world" />
+    <!-- <link name="world" /> -->
   <link name="person">
     <visual>
@@ -36,5 +36,5 @@
     <xacro:default_inertial mass="70"/>
   </link>
-  <joint name="world_to_person" type="prismatic">
+  <!-- <joint name="world_to_person" type="prismatic">
     <axis xyz="1 0 0"/>
     <limit lower="-3" upper="2" velocity="100" effort="100"/>
@@ -42,4 +42,4 @@
     <child link="person"/>
     <origin xyz="${xyz}" />
-  </joint>
+  </joint> -->
 </robot>

File: ros_1/catkin_ws/src/my_package/urdf/table.xacro (robot description, xacro)
@@ -2,5 +2,5 @@
 <robot name="table" xmlns:xacro="http://ros.org/wiki/xacro">
     <!-- o_x is the position of the table of the table along x axis -->
-    <xacro:property name="o_x" value="0.5" />
+    <xacro:property name="o_x" value="0.1" />
     <!-- o_y is the position of the table of the table along y axis -->
     <xacro:property name="o_y" value="-0.7" />
