Commit message: Update

File: ros_1/catkin_ws/src/my_package/urdf/person_new.xacro (robot description, xacro)
@@ -1,5 +1,5 @@
 <?xml version="1.0"?>
 <robot name="person" xmlns:xacro="http://ros.org/wiki/xacro">
-  <xacro:property name="xyz" value="2 2 0" />
+  <xacro:property name="xyz" value="1.2 0 0" />
     <xacro:property name="person_width_x" value="0.3" />
     <xacro:property name="person_width_y" value="0.5" />

Commit message: Update

File: ros_1/catkin_ws/src/my_package/urdf/person_new.xacro (robot description, xacro)
@@ -1,5 +1,5 @@
 <?xml version="1.0"?>
 <robot name="person" xmlns:xacro="http://ros.org/wiki/xacro">
-  <xacro:property name="xyz" value="1.2 0 0" />
+  <xacro:property name="xyz" value="1.0 0 0" />
     <xacro:property name="person_width_x" value="0.3" />
     <xacro:property name="person_width_y" value="0.5" />

Commit message: Update

File: ros_1/catkin_ws/src/my_package/urdf/person_new.xacro (robot description, xacro)
@@ -1,5 +1,5 @@
 <?xml version="1.0"?>
 <robot name="person" xmlns:xacro="http://ros.org/wiki/xacro">
-  <xacro:property name="xyz" value="1.0 0 0" />
+  <xacro:property name="xyz" value="1.2 0 0" />
     <xacro:property name="person_width_x" value="0.2" />
     <xacro:property name="person_width_y" value="0.2" />
