Commit message: colors updated

File: ros_1/catkin_ws/src/my_package/urdf/dirt_box.xacro (robot description, xacro)
@@ -33,5 +33,5 @@
   </joint>
   <gazebo reference="$(arg dirt_box_name)">
-    <material>Gazebo/Black</material>
+    <material>Gazebo/DarkGray</material>
     <mu1>0.2</mu1>
     <mu2>0.2</mu2>

Commit message: dirty updated

File: ros_1/catkin_ws/src/my_package/urdf/dirt_box.xacro (robot description, xacro)
@@ -33,5 +33,5 @@
   </joint>
   <gazebo reference="$(arg dirt_box_name)">
-    <material>Gazebo/DarkGray</material>
+    <material>Gazebo/Black</material>
     <mu1>0.2</mu1>
     <mu2>0.2</mu2>
